File: manuform.pcb.kicad_sch (KiCad schematic)
At the start: 8 parts, among them J1 Conn_01x04, J2 Conn_01x04, J3 Conn_01x04, SW1 SW_DIP_x01, SW2 SW_DIP_x01, SW3 SW_DIP_x01, SW4 SW_DIP_x01

Commit message: added MX diodeless switches.
Parts:
- SW1, SW2, SW3, SW4: footprint switchCustom:SW_Kailh_Choc_V2_elongated -> switchCustom:SW_Cherry_MX_1.00u_PCB
Changed lines of the file:
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@@
       (effects (font (size 1.27 1.27)))
     )
-    (property "Footprint" "switchCustom:SW_Kailh_Choc_V2_elongated" (at 111.76 64.77 0)
+    (property "Footprint" "switchCustom:SW_Cherry_MX_1.00u_PCB" (at 111.76 64.77 0)
       (effects (font (size 1.27 1.27)) hide)
     )
@@
       (effects (font (size 1.27 1.27)))
     )
-    (property "Footprint" "switchCustom:SW_Kailh_Choc_V2_elongated" (at 111.76 76.2 0)
+    (property "Footprint" "switchCustom:SW_Cherry_MX_1.00u_PCB" (at 111.76 76.2 0)
       (effects (font (size 1.27 1.27)) hide)
     )
@@
       (effects (font (size 1.27 1.27)))
     )
-    (property "Footprint" "switchCustom:SW_Kailh_Choc_V2_elongated" (at 111.76 53.34 0)
+    (property "Footprint" "switchCustom:SW_Cherry_MX_1.00u_PCB" (at 111.76 53.34 0)
       (effects (font (size 1.27 1.27)) hide)
     )
@@
       (effects (font (size 1.27 1.27)))
     )
-    (property "Footprint" "switchCustom:SW_Kailh_Choc_V2_elongated" (at 111.76 87.63 0)
+    (property "Footprint" "switchCustom:SW_Cherry_MX_1.00u_PCB" (at 111.76 87.63 0)
       (effects (font (size 1.27 1.27)) hide)
     )
